File: Electrical/NVR.kicad_sch (KiCad schematic)
At the start: 6 parts

Commit message: switch to 20V PD input
Other:
- removed sheet Secure Enclave
- sheet LattePanda Module ports: added none; removed I2C_SCL_2, I2C_SDA_2
Changed lines of the file:
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@@
 	(wire
 		(pts
-			(xy 341.63 154.94) (xy 363.22 154.94)
-		)
-		(stroke
-			(width 0)
-			(type default)
-		)
-	)
-	(wire
-		(pts
 			(xy 194.31 297.18) (xy 227.33 297.18)
 		)
@@
 	(wire
 		(pts
-			(xy 341.63 152.4) (xy 363.22 152.4)
-		)
-		(stroke
-			(width 0)
-			(type default)
-		)
-	)
-	(wire
-		(pts
 			(xy 341.63 123.19) (xy 363.22 123.19)
 		)
@@
 			)
 		)
-		(pin "I2C_SDA_2" bidirectional
-			(at 341.63 154.94 0)
-			(effects
-				(font
-					(size 1.27 1.27)
-				)
-				(justify right)
-			)
-		)
-		(pin "I2C_SCL_2" output
-			(at 341.63 152.4 0)
-			(effects
-				(font
-					(size 1.27 1.27)
-				)
-				(justify right)
-			)
-		)
 		(pin "SPI-CS" bidirectional
 			(at 227.33 156.21 180)
@@
 				)
 			)
-		)
-	)
-	(sheet
-		(at 363.22 146.05)
-		(size 27.94 17.78)
-		(exclude_from_sim no)
-		(in_bom yes)
-		(on_board yes)
-		(dnp no)
-		(fields_autoplaced yes)
-		(stroke
-			(width 0.1524)
-			(type solid)
-		)
-		(fill
-			(color 0 0 0 0.0000)
-		)
-		(property "Sheetname" "Secure Enclave"
-			(at 363.22 145.3384 0)
-			(effects
-				(font
-					(size 1.27 1.27)
-				)
-				(justify left bottom)
-			)
-		)
-		(property "Sheetfile" "Security.kicad_sch"
-			(at 363.22 164.4146 0)
-			(effects
-				(font
-					(size 1.27 1.27)
-				)
-				(justify left top)
-			)
-		)
-		(property "Field2" ""
-			(at 363.22 146.05 0)
-			(effects
-				(font
-					(size 1.27 1.27)
-				)
-			)
-		)
-		(pin "I2C_SCL_2" input
-			(at 363.22 152.4 180)
-			(effects
-				(font
-					(size 1.27 1.27)
-				)
-				(justify left)
-			)
-		)
-		(pin "I2C_SDA_2" bidirectional
-			(at 363.22 154.94 180)
-			(effects
-				(font
-					(size 1.27 1.27)
-				)
-				(justify left)
-			)
-		)
-		(instances
-			(project "NVR"
-				(path "/2a6d114a-7fd7-4207-b5f7-4ea9c34f36aa"
-					(page "11")
-				)
-			)
