File: Electrical/PSU.kicad_sch (KiCad schematic)
At the start: 112 parts, among them IC2 SiC437AED-T1-GE3, J15 Conn_01x03_Pin, J16 USB_C_Receptacle_USB2.0, Q10 2N7002, Q8 2N7002, Q9 2N7002, SW1 SW_Push, U13 HT7533, U14 CH224Q_C46061833, U15 SY8253ADC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

Commit message: Update Board According to DFA Review
Updated Ethernet Jack
Updated L3 Inductor
Fixed a few errors
Updated mounting hole size
Parts:
- U10, U9: value ~ -> (none)

Commit message: further changes required by DFA review
Parts:
- C145, C146, C147, C148: footprint A_HDJ_Library:C_0402_1005Metric -> Capacitor_SMD:C_0603_1608Metric
- D24: footprint Diode_SMD:D_SOD-323 -> Diode_SMD:D_SOD-923
- L1, L2, L4, L5: footprint A_HDJ_Library:L_Sunlord_SWPA4020S -> inductor-2:SPM4010-4020
Changed lines of the file:
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@@
 			)
 		)
-		(property "Footprint" "Diode_SMD:D_SOD-323"
+		(property "Footprint" "Diode_SMD:D_SOD-923"
 			(at 458.47 228.6 0)
 			(hide yes)
@@
 			)
 		)
-		(property "Footprint" "A_HDJ_Library:C_0402_1005Metric"
+		(property "Footprint" "Capacitor_SMD:C_0603_1608Metric"
 			(at 445.4652 176.53 0)
 			(hide yes)
@@
 			)
 		)
-		(property "Footprint" "A_HDJ_Library:L_Sunlord_SWPA4020S"
+		(property "Footprint" "inductor-2:SPM4010-4020"
 			(at 299.72 350.52 0)
 			(hide yes)
@@
 			)
 		)
-		(property "Footprint" "A_HDJ_Library:C_0402_1005Metric"
+		(property "Footprint" "Capacitor_SMD:C_0603_1608Metric"
 			(at 435.3052 176.53 0)
 			(hide yes)
@@
 			)
 		)
-		(property "Footprint" "A_HDJ_Library:L_Sunlord_SWPA4020S"
+		(property "Footprint" "inductor-2:SPM4010-4020"
 			(at 314.96 229.87 0)
 			(hide yes)
@@
 			)
 		)
-		(property "Footprint" "A_HDJ_Library:C_0402_1005Metric"
+		(property "Footprint" "Capacitor_SMD:C_0603_1608Metric"
 			(at 440.3852 176.53 0)
 			(hide yes)
@@
 			)
 		)
-		(property "Footprint" "A_HDJ_Library:L_Sunlord_SWPA4020S"
+		(property "Footprint" "inductor-2:SPM4010-4020"
 			(at 501.65 278.13 0)
 			(hide yes)
@@
 			)
 		)
-		(property "Footprint" "A_HDJ_Library:L_Sunlord_SWPA4020S"
+		(property "Footprint" "inductor-2:SPM4010-4020"
 			(at 501.65 240.03 0)
 			(hide yes)
@@
 			)
 		)
-		(property "Footprint" "A_HDJ_Library:C_0402_1005Metric"
+		(property "Footprint" "Capacitor_SMD:C_0603_1608Metric"
 			(at 450.5452 176.53 0)
 			(hide yes)
